File: Neopixel/Neopixel.kicad_pcb (KiCad board)
At the start: 2 copper layers, 105 x 105 mm, 70 parts

Commit message: designing
Parts:
- added C1: 220uF, Capacitor_SMD:C_1206_3216Metric, F.Cu at (19.5, 33.0)
- renumbered Din to DIn, Dout to DOut
Routing:
- net GND: track 719.8 -> 722.3 mm
- net +5V: track 696.6 -> 698.7 mm
