File: Neopixel/Neopixel.kicad_sch (KiCad schematic)
At the start: 1 part

Commit message: designing
Parts:
- added D10, D11, D12, D13, D14, D15, D16, D17, D18, D19, D2, D20, D21, D22, D23, D24, D25, D26, D27, D28, D3, D4, D5, D6, D7, D8, D9: WS2812B, LED_SMD:LED_WS2812B_PLCC4_5.0x5.0mm_P3.2mm, symbol LED:WS2812B
Connections:
- net +5V: now also D10.1 (VDD), D11.1 (VDD), D12.1 (VDD), D13.1 (VDD), D14.1 (VDD), D15.1 (VDD), D16.1 (VDD), D17.1 (VDD), D18.1 (VDD), D19.1 (VDD), D2.1 (VDD), D20.1 (VDD), D21.1 (VDD), D22.1 (VDD), D23.1 (VDD), D24.1 (VDD), D25.1 (VDD), D26.1 (VDD), D27.1 (VDD), D28.1 (VDD), D3.1 (VDD), D4.1 (VDD), D5.1 (VDD), D6.1 (VDD), D7.1 (VDD), D8.1 (VDD), D9.1 (VDD)
- net GND: now also D10.3 (VSS), D11.3 (VSS), D12.3 (VSS), D13.3 (VSS), D14.3 (VSS), D15.3 (VSS), D16.3 (VSS), D17.3 (VSS), D18.3 (VSS), D19.3 (VSS), D2.3 (VSS), D20.3 (VSS), D21.3 (VSS), D22.3 (VSS), D23.3 (VSS), D24.3 (VSS), D25.3 (VSS), D26.3 (VSS), D27.3 (VSS), D28.3 (VSS), D3.3 (VSS), D4.3 (VSS), D5.3 (VSS), D6.3 (VSS), D7.3 (VSS), D8.3 (VSS), D9.3 (VSS)
- net at D1.2 (DOUT): now also D2.4 (DIN)
- new net: D25.2 (DOUT), D26.4 (DIN)
- new net: D24.2 (DOUT), D25.4 (DIN)
- new net: D21.2 (DOUT), D22.4 (DIN)
- new net: D20.2 (DOUT), D21.4 (DIN)
- new net: D6.2 (DOUT), D7.4 (DIN)
- new net: D5.2 (DOUT), D6.4 (DIN)
- new net: D4.2 (DOUT), D5.4 (DIN)
- new net: D8.2 (DOUT), D9.4 (DIN)
- new net: D7.2 (DOUT), D8.4 (DIN)
- new net: D13.2 (DOUT), D14.4 (DIN)
- new net: D12.2 (DOUT), D13.4 (DIN)
- new net: D11.2 (DOUT), D12.4 (DIN)
- new net: D10.2 (DOUT), D11.4 (DIN)
- new net: D22.2 (DOUT), D23.4 (DIN)
- new net: D3.2 (DOUT), D4.4 (DIN)
- new net: D28.2 (DOUT), D3.4 (DIN)
- new net: D27.2 (DOUT), D28.4 (DIN)
- new net: D2.2 (DOUT), D27.4 (DIN)
- new net: D23.2 (DOUT), D24.4 (DIN)
- new net: D10.4 (DIN), D9.2 (DOUT)
- new net: D17.2 (DOUT), D18.4 (DIN)
- new net: D16.2 (DOUT), D17.4 (DIN)
- new net: D15.2 (DOUT), D16.4 (DIN)
- new net: D14.2 (DOUT), D15.4 (DIN)
- new net: D19.2 (DOUT), D20.4 (DIN)
- new net: D18.2 (DOUT), D19.4 (DIN)

Commit message: designing
Parts:
- added TP1, TP10, TP11, TP12, TP13, TP14, TP15, TP16, TP17, TP18, TP19, TP2, TP20, TP21, TP22, TP23, TP24, TP25, TP26, TP27, TP28, TP29, TP3, TP30, TP31, TP32, TP33, TP34, TP35, TP36, TP37, TP38, TP39, TP4, TP40, TP41, TP42, TP43, TP44, TP45, TP46, TP47, TP48, TP49, TP5, TP50, TP51, TP52, TP53, TP54, TP55, TP56, TP57, TP58, TP59, TP6, TP60, TP61, TP62, TP63, TP64, TP65, TP66, TP67, TP68, TP69, TP7, TP70, TP71, TP72, TP73, TP74, TP75, TP76, TP77, TP78, TP79, TP8, TP80, TP81, TP82, TP83, TP84, TP9: TestPoint, Pegoku:TestPoint, symbol Connector:TestPoint
Connections:
- net +5V: now also TP11.1, TP14.1, TP17.1, TP2.1, TP20.1, TP23.1, TP26.1, TP29.1, TP32.1, TP35.1, TP38.1, TP41.1, TP44.1, TP47.1, TP5.1, TP50.1, TP53.1, TP56.1, TP59.1, TP62.1, TP65.1, TP68.1, TP71.1, TP74.1, TP77.1, TP8.1, TP80.1, TP83.1
- net GND: now also TP10.1, TP13.1, TP16.1, TP19.1, TP22.1, TP25.1, TP28.1, TP3.1, TP31.1, TP34.1, TP37.1, TP4.1, TP40.1, TP43.1, TP46.1, TP49.1, TP52.1, TP55.1, TP58.1, TP61.1, TP64.1, TP67.1, TP7.1, TP70.1, TP73.1, TP76.1, TP79.1, TP82.1
- net at D1.4 (DIN): now also TP1.1

Commit message: designing
Parts:
- removed D17, D18, D19, D20, D21, D22, D23, D24, D25, D26, D27, D28: WS2812B, LED_SMD:LED_WS2812B_PLCC4_5.0x5.0mm_P3.2mm, symbol LED:WS2812B
- removed TP10, TP11, TP12, TP13, TP14, TP15, TP16, TP17, TP18, TP19, TP20, TP21, TP22, TP23, TP24, TP25, TP26, TP27, TP28, TP29, TP30, TP31, TP32, TP33, TP34, TP35, TP36, TP37, TP38, TP39, TP4, TP40, TP41, TP42, TP43, TP44, TP45, TP46, TP47, TP48, TP49, TP5, TP50, TP51, TP52, TP53, TP54, TP55, TP56, TP57, TP58, TP59, TP6, TP60, TP61, TP62, TP63, TP64, TP65, TP66, TP67, TP68, TP69, TP7, TP70, TP71, TP72, TP73, TP74, TP75, TP76, TP77, TP78, TP79, TP8, TP80, TP81, TP82, TP83, TP84, TP9: TestPoint, Pegoku:TestPoint, symbol Connector:TestPoint
Connections:
- net at D3.4 (DIN): now also D2.2 (DOUT)

Commit message: designing
Parts:
- added D100, D101, D102, D103, D104, D105, D106, D107, D108, D109, D110, D111, D112, D113, D114, D115, D116, D117, D118, D119, D120, D121, D122, D123, D124, D125, D126, D127, D128, D129, D130, D131, D132, D133, D134, D135, D136, D137, D138, D139, D140, D141, D142, D143, D144, D145, D146, D147, D148, D149, D150, D151, D152, D153, D154, D155, D156, D157, D158, D159, D160, D161, D162, D163, D164, D165, D166, D167, D168, D169, D17, D170, D171, D172, D173, D174, D175, D176, D177, D178, D179, D18, D180, D181, D182, D183, D184, D185, D186, D187, D188, D189, D19, D190, D191, D192, D193, D194, D195, D196, D197, D198, D199, D20, D200, D201, D202, D203, D204, D205, D206, D207, D208, D209, D21, D210, D211, D212, D213, D214, D215, D216, D217, D218, D219, D22, D220, D221, D222, D223, D224, D225, D226, D227, D228, D229, D23, D230, D231, D232, D233, D234, D235, D236, D237, D238, D239, D24, D240, D241, D242, D243, D244, D245, D246, D247, D248, D249, D25, D250, D251, D252, D253, D254, D255, D256, D26, D27, D28, D29, D30, D31, D32, D33, D34, D35, D36, D37, D38, D39, D40, D41, D42, D43, D44, D45, D46, D47, D48, D49, D50, D51, D52, D53, D54, D55, D56, D57, D58, D59, D60, D61, D62, D63, D64, D65, D66, D67, D68, D69, D70, D71, D72, D73, D74, D75, D76, D77, D78, D79, D80, D81, D82, D83, D84, D85, D86, D87, D88, D89, D90, D91, D92, D93, D94, D95, D96, D97, D98, D99: WS2812B, LED_SMD:LED_WS2812B_PLCC4_5.0x5.0mm_P3.2mm, symbol LED:WS2812B
Connections:
- net +5V: now also D100.1 (VDD), D101.1 (VDD), D102.1 (VDD), D103.1 (VDD), D104.1 (VDD), D105.1 (VDD), D106.1 (VDD), D107.1 (VDD), D108.1 (VDD), D109.1 (VDD), D110.1 (VDD), D111.1 (VDD), D112.1 (VDD), D113.1 (VDD), D114.1 (VDD), D115.1 (VDD), D116.1 (VDD), D117.1 (VDD), D118.1 (VDD), D119.1 (VDD), D120.1 (VDD), D121.1 (VDD), D122.1 (VDD), D123.1 (VDD), D124.1 (VDD), D125.1 (VDD), D126.1 (VDD), D127.1 (VDD), D128.1 (VDD), D129.1 (VDD), D130.1 (VDD), D131.1 (VDD), D132.1 (VDD), D133.1 (VDD), D134.1 (VDD), D135.1 (VDD), D136.1 (VDD), D137.1 (VDD), D138.1 (VDD), D139.1 (VDD), D140.1 (VDD), D141.1 (VDD), D142.1 (VDD), D143.1 (VDD), D144.1 (VDD), D145.1 (VDD), D146.1 (VDD), D147.1 (VDD), D148.1 (VDD), D149.1 (VDD), D150.1 (VDD), D151.1 (VDD), D152.1 (VDD), D153.1 (VDD), D154.1 (VDD), D155.1 (VDD), D156.1 (VDD), D157.1 (VDD), D158.1 (VDD), D159.1 (VDD), D160.1 (VDD), D161.1 (VDD), D162.1 (VDD), D163.1 (VDD), D164.1 (VDD), D165.1 (VDD), D166.1 (VDD), D167.1 (VDD), D168.1 (VDD), D169.1 (VDD), D17.1 (VDD), D170.1 (VDD), D171.1 (VDD), D172.1 (VDD), D173.1 (VDD), D174.1 (VDD), D175.1 (VDD), D176.1 (VDD), D177.1 (VDD), D178.1 (VDD), D179.1 (VDD), D18.1 (VDD), D180.1 (VDD), D181.1 (VDD), D182.1 (VDD), D183.1 (VDD), D184.1 (VDD), D185.1 (VDD), D186.1 (VDD), D187.1 (VDD), D188.1 (VDD), D189.1 (VDD), D19.1 (VDD), D190.1 (VDD), D191.1 (VDD), D192.1 (VDD), D193.1 (VDD), D194.1 (VDD), D195.1 (VDD), D196.1 (VDD), D197.1 (VDD), D198.1 (VDD), D199.1 (VDD), D20.1 (VDD), D200.1 (VDD), D201.1 (VDD), D202.1 (VDD), D203.1 (VDD), D204.1 (VDD), D205.1 (VDD), D206.1 (VDD), D207.1 (VDD), D208.1 (VDD), D209.1 (VDD), D21.1 (VDD), D210.1 (VDD), D211.1 (VDD), D212.1 (VDD), D213.1 (VDD), D214.1 (VDD), D215.1 (VDD), D216.1 (VDD), D217.1 (VDD), D218.1 (VDD), D219.1 (VDD), D22.1 (VDD), D220.1 (VDD), D221.1 (VDD), D222.1 (VDD), D223.1 (VDD), D224.1 (VDD), D225.1 (VDD), D226.1 (VDD), D227.1 (VDD), D228.1 (VDD), D229.1 (VDD), D23.1 (VDD), D230.1 (VDD), D231.1 (VDD), D232.1 (VDD), D233.1 (VDD), D234.1 (VDD), D235.1 (VDD), D236.1 (VDD), D237.1 (VDD), D238.1 (VDD), D239.1 (VDD), D24.1 (VDD), D240.1 (VDD), D241.1 (VDD), D242.1 (VDD), D243.1 (VDD), D244.1 (VDD), D245.1 (VDD), D246.1 (VDD), D247.1 (VDD), D248.1 (VDD), D249.1 (VDD), D25.1 (VDD), D250.1 (VDD), D251.1 (VDD), D252.1 (VDD), D253.1 (VDD), D254.1 (VDD), D255.1 (VDD), D256.1 (VDD), D26.1 (VDD), D27.1 (VDD), D28.1 (VDD), D29.1 (VDD), D30.1 (VDD), D31.1 (VDD), D32.1 (VDD), D33.1 (VDD), D34.1 (VDD), D35.1 (VDD), D36.1 (VDD), D37.1 (VDD), D38.1 (VDD), D39.1 (VDD), D40.1 (VDD), D41.1 (VDD), D42.1 (VDD), D43.1 (VDD), D44.1 (VDD), D45.1 (VDD), D46.1 (VDD), D47.1 (VDD), D48.1 (VDD), D49.1 (VDD), D50.1 (VDD), D51.1 (VDD), D52.1 (VDD), D53.1 (VDD), D54.1 (VDD), D55.1 (VDD), D56.1 (VDD), D57.1 (VDD), D58.1 (VDD), D59.1 (VDD), D60.1 (VDD), D61.1 (VDD), D62.1 (VDD), D63.1 (VDD), D64.1 (VDD), D65.1 (VDD), D66.1 (VDD), D67.1 (VDD), D68.1 (VDD), D69.1 (VDD), D70.1 (VDD), D71.1 (VDD), D72.1 (VDD), D73.1 (VDD), D74.1 (VDD), D75.1 (VDD), D76.1 (VDD), D77.1 (VDD), D78.1 (VDD), D79.1 (VDD), D80.1 (VDD), D81.1 (VDD), D82.1 (VDD), D83.1 (VDD), D84.1 (VDD), D85.1 (VDD), D86.1 (VDD), D87.1 (VDD), D88.1 (VDD), D89.1 (VDD), D90.1 (VDD), D91.1 (VDD), D92.1 (VDD), D93.1 (VDD), D94.1 (VDD), D95.1 (VDD), D96.1 (VDD), D97.1 (VDD), D98.1 (VDD), D99.1 (VDD)
- net GND: now also D100.3 (VSS), D101.3 (VSS), D102.3 (VSS), D103.3 (VSS), D104.3 (VSS), D105.3 (VSS), D106.3 (VSS), D107.3 (VSS), D108.3 (VSS), D109.3 (VSS), D110.3 (VSS), D111.3 (VSS), D112.3 (VSS), D113.3 (VSS), D114.3 (VSS), D115.3 (VSS), D116.3 (VSS), D117.3 (VSS), D118.3 (VSS), D119.3 (VSS), D120.3 (VSS), D121.3 (VSS), D122.3 (VSS), D123.3 (VSS), D124.3 (VSS), D125.3 (VSS), D126.3 (VSS), D127.3 (VSS), D128.3 (VSS), D129.3 (VSS), D130.3 (VSS), D131.3 (VSS), D132.3 (VSS), D133.3 (VSS), D134.3 (VSS), D135.3 (VSS), D136.3 (VSS), D137.3 (VSS), D138.3 (VSS), D139.3 (VSS), D140.3 (VSS), D141.3 (VSS), D142.3 (VSS), D143.3 (VSS), D144.3 (VSS), D145.3 (VSS), D146.3 (VSS), D147.3 (VSS), D148.3 (VSS), D149.3 (VSS), D150.3 (VSS), D151.3 (VSS), D152.3 (VSS), D153.3 (VSS), D154.3 (VSS), D155.3 (VSS), D156.3 (VSS), D157.3 (VSS), D158.3 (VSS), D159.3 (VSS), D160.3 (VSS), D161.3 (VSS), D162.3 (VSS), D163.3 (VSS), D164.3 (VSS), D165.3 (VSS), D166.3 (VSS), D167.3 (VSS), D168.3 (VSS), D169.3 (VSS), D17.3 (VSS), D170.3 (VSS), D171.3 (VSS), D172.3 (VSS), D173.3 (VSS), D174.3 (VSS), D175.3 (VSS), D176.3 (VSS), D177.3 (VSS), D178.3 (VSS), D179.3 (VSS), D18.3 (VSS), D180.3 (VSS), D181.3 (VSS), D182.3 (VSS), D183.3 (VSS), D184.3 (VSS), D185.3 (VSS), D186.3 (VSS), D187.3 (VSS), D188.3 (VSS), D189.3 (VSS), D19.3 (VSS), D190.3 (VSS), D191.3 (VSS), D192.3 (VSS), D193.3 (VSS), D194.3 (VSS), D195.3 (VSS), D196.3 (VSS), D197.3 (VSS), D198.3 (VSS), D199.3 (VSS), D20.3 (VSS), D200.3 (VSS), D201.3 (VSS), D202.3 (VSS), D203.3 (VSS), D204.3 (VSS), D205.3 (VSS), D206.3 (VSS), D207.3 (VSS), D208.3 (VSS), D209.3 (VSS), D21.3 (VSS), D210.3 (VSS), D211.3 (VSS), D212.3 (VSS), D213.3 (VSS), D214.3 (VSS), D215.3 (VSS), D216.3 (VSS), D217.3 (VSS), D218.3 (VSS), D219.3 (VSS), D22.3 (VSS), D220.3 (VSS), D221.3 (VSS), D222.3 (VSS), D223.3 (VSS), D224.3 (VSS), D225.3 (VSS), D226.3 (VSS), D227.3 (VSS), D228.3 (VSS), D229.3 (VSS), D23.3 (VSS), D230.3 (VSS), D231.3 (VSS), D232.3 (VSS), D233.3 (VSS), D234.3 (VSS), D235.3 (VSS), D236.3 (VSS), D237.3 (VSS), D238.3 (VSS), D239.3 (VSS), D24.3 (VSS), D240.3 (VSS), D241.3 (VSS), D242.3 (VSS), D243.3 (VSS), D244.3 (VSS), D245.3 (VSS), D246.3 (VSS), D247.3 (VSS), D248.3 (VSS), D249.3 (VSS), D25.3 (VSS), D250.3 (VSS), D251.3 (VSS), D252.3 (VSS), D253.3 (VSS), D254.3 (VSS), D255.3 (VSS), D256.3 (VSS), D26.3 (VSS), D27.3 (VSS), D28.3 (VSS), D29.3 (VSS), D30.3 (VSS), D31.3 (VSS), D32.3 (VSS), D33.3 (VSS), D34.3 (VSS), D35.3 (VSS), D36.3 (VSS), D37.3 (VSS), D38.3 (VSS), D39.3 (VSS), D40.3 (VSS), D41.3 (VSS), D42.3 (VSS), D43.3 (VSS), D44.3 (VSS), D45.3 (VSS), D46.3 (VSS), D47.3 (VSS), D48.3 (VSS), D49.3 (VSS), D50.3 (VSS), D51.3 (VSS), D52.3 (VSS), D53.3 (VSS), D54.3 (VSS), D55.3 (VSS), D56.3 (VSS), D57.3 (VSS), D58.3 (VSS), D59.3 (VSS), D60.3 (VSS), D61.3 (VSS), D62.3 (VSS), D63.3 (VSS), D64.3 (VSS), D65.3 (VSS), D66.3 (VSS), D67.3 (VSS), D68.3 (VSS), D69.3 (VSS), D70.3 (VSS), D71.3 (VSS), D72.3 (VSS), D73.3 (VSS), D74.3 (VSS), D75.3 (VSS), D76.3 (VSS), D77.3 (VSS), D78.3 (VSS), D79.3 (VSS), D80.3 (VSS), D81.3 (VSS), D82.3 (VSS), D83.3 (VSS), D84.3 (VSS), D85.3 (VSS), D86.3 (VSS), D87.3 (VSS), D88.3 (VSS), D89.3 (VSS), D90.3 (VSS), D91.3 (VSS), D92.3 (VSS), D93.3 (VSS), D94.3 (VSS), D95.3 (VSS), D96.3 (VSS), D97.3 (VSS), D98.3 (VSS), D99.3 (VSS)
- net at D16.2 (DOUT): now also D17.4 (DIN)
- new net: D191.2 (DOUT), D193.4 (DIN)
- new net: D189.2 (DOUT), D191.4 (DIN)
- new net: D130.4 (DIN), D132.2 (DOUT)
- new net: D132.4 (DIN), D134.2 (DOUT)
- new net: D76.2 (DOUT), D77.4 (DIN)
- new net: D75.2 (DOUT), D76.4 (DIN)
- new net: D203.2 (DOUT), D205.4 (DIN)
- new net: D201.2 (DOUT), D203.4 (DIN)
- new net: D106.2 (DOUT), D107.4 (DIN)
- new net: D105.2 (DOUT), D106.4 (DIN)
- new net: D46.2 (DOUT), D47.4 (DIN)
- new net: D45.2 (DOUT), D46.4 (DIN)
- new net: D242.4 (DIN), D244.2 (DOUT)
- new net: D244.4 (DIN), D246.2 (DOUT)
- new net: D51.2 (DOUT), D52.4 (DIN)
- new net: D50.2 (DOUT), D51.4 (DIN)
- new net: D100.4 (DIN), D99.2 (DOUT)
- new net: D98.2 (DOUT), D99.4 (DIN)
- new net: D111.2 (DOUT), D112.4 (DIN)
- new net: D110.2 (DOUT), D111.4 (DIN)
- new net: D56.2 (DOUT), D57.4 (DIN)
- new net: D55.2 (DOUT), D56.4 (DIN)
- new net: D157.2 (DOUT), D159.4 (DIN)
- new net: D155.2 (DOUT), D157.4 (DIN)
- new net: D69.2 (DOUT), D70.4 (DIN)
- new net: D68.2 (DOUT), D69.4 (DIN)
- new net: D121.2 (DOUT), D122.4 (DIN)
- new net: D120.2 (DOUT), D121.4 (DIN)
- new net: D77.2 (DOUT), D78.4 (DIN)
- new net: D146.4 (DIN), D148.2 (DOUT)
- new net: D148.4 (DIN), D150.2 (DOUT)
- new net: D197.2 (DOUT), D199.4 (DIN)
- new net: D195.2 (DOUT), D197.4 (DIN)
- new net: D108.2 (DOUT), D109.4 (DIN)
- new net: D107.2 (DOUT), D108.4 (DIN)
- new net: D166.4 (DIN), D168.2 (DOUT)
- new net: D168.4 (DIN), D170.2 (DOUT)
- new net: D66.2 (DOUT), D67.4 (DIN)
- new net: D65.2 (DOUT), D66.4 (DIN)
- new net: D241.2 (DOUT), D243.4 (DIN)
- new net: D239.2 (DOUT), D241.4 (DIN)
- new net: D214.4 (DIN), D216.2 (DOUT)
- new net: D216.4 (DIN), D218.2 (DOUT)
- new net: D22.2 (DOUT), D23.4 (DIN)
- new net: D21.2 (DOUT), D22.4 (DIN)
- new net: D89.2 (DOUT), D90.4 (DIN)
- new net: D88.2 (DOUT), D89.4 (DIN)
- new net: D231.2 (DOUT), D233.4 (DIN)
- new net: D229.2 (DOUT), D231.4 (DIN)
- new net: D67.2 (DOUT), D68.4 (DIN)
- new net: D212.4 (DIN), D214.2 (DOUT)
- new net: D176.4 (DIN), D178.2 (DOUT)
- new net: D178.4 (DIN), D180.2 (DOUT)
- new net: D63.2 (DOUT), D64.4 (DIN)
- new net: D62.2 (DOUT), D63.4 (DIN)
- new net: D18.2 (DOUT), D19.4 (DIN)
- new net: D17.2 (DOUT), D18.4 (DIN)
- new net: D198.4 (DIN), D200.2 (DOUT)
- new net: D200.4 (DIN), D202.2 (DOUT)
- new net: D134.4 (DIN), D136.2 (DOUT)
- new net: D136.4 (DIN), D138.2 (DOUT)
- new net: D238.4 (DIN), D240.2 (DOUT)
- new net: D240.4 (DIN), D242.2 (DOUT)
- new net: D41.2 (DOUT), D42.4 (DIN)
- new net: D40.2 (DOUT), D41.4 (DIN)
- new net: D233.2 (DOUT), D235.4 (DIN)
- new net: D139.2 (DOUT), D141.4 (DIN)
- new net: D137.2 (DOUT), D139.4 (DIN)
- new net: D179.2 (DOUT), D181.4 (DIN)
- new net: D177.2 (DOUT), D179.4 (DIN)
- new net: D125.2 (DOUT), D126.4 (DIN)
- new net: D124.2 (DOUT), D125.4 (DIN)
- new net: D131.2 (DOUT), D133.4 (DIN)
- new net: D129.2 (DOUT), D131.4 (DIN)
- new net: D253.2 (DOUT), D255.4 (DIN)
- new net: D251.2 (DOUT), D253.4 (DIN)
- new net: D249.2 (DOUT), D251.4 (DIN)
- new net: D207.2 (DOUT), D209.4 (DIN)
- new net: D205.2 (DOUT), D207.4 (DIN)
- new net: D47.2 (DOUT), D48.4 (DIN)
- new net: D38.2 (DOUT), D39.4 (DIN)
- new net: D37.2 (DOUT), D38.4 (DIN)
- new net: D20.2 (DOUT), D21.4 (DIN)
- new net: D199.2 (DOUT), D201.4 (DIN)
- new net: D192.4 (DIN), D194.2 (DOUT)
- new net: D194.4 (DIN), D196.2 (DOUT)
- new net: D254.4 (DIN), D256.2 (DOUT)
- new net: D255.2 (DOUT), D256.4 (DIN)
- new net: D19.2 (DOUT), D20.4 (DIN)
- new net: D103.2 (DOUT), D104.4 (DIN)
- new net: D102.2 (DOUT), D103.4 (DIN)
- new net: D44.2 (DOUT), D45.4 (DIN)
- new net: D87.2 (DOUT), D88.4 (DIN)
- new net: D163.2 (DOUT), D165.4 (DIN)
- new net: D161.2 (DOUT), D163.4 (DIN)
- new net: D220.4 (DIN), D222.2 (DOUT)
- new net: D222.4 (DIN), D224.2 (DOUT)
- new net: D171.2 (DOUT), D173.4 (DIN)
- new net: D169.2 (DOUT), D171.4 (DIN)
- new net: D226.4 (DIN), D228.2 (DOUT)
- new net: D228.4 (DIN), D230.2 (DOUT)
- new net: D83.2 (DOUT), D84.4 (DIN)
- new net: D82.2 (DOUT), D83.4 (DIN)
- new net: D33.2 (DOUT), D34.4 (DIN)
- new net: D32.2 (DOUT), D33.4 (DIN)
- new net: D159.2 (DOUT), D161.4 (DIN)
- new net: D127.2 (DOUT), D128.4 (DIN)
- new net: D126.2 (DOUT), D127.4 (DIN)
- new net: D27.2 (DOUT), D28.4 (DIN)
- new net: D26.2 (DOUT), D27.4 (DIN)
- new net: D149.2 (DOUT), D151.4 (DIN)
- new net: D147.2 (DOUT), D149.4 (DIN)
- new net: D237.2 (DOUT), D239.4 (DIN)
- new net: D235.2 (DOUT), D237.4 (DIN)
- new net: D86.2 (DOUT), D87.4 (DIN)
- new net: D170.4 (DIN), D172.2 (DOUT)
- new net: D172.4 (DIN), D174.2 (DOUT)
- new net: D96.2 (DOUT), D97.4 (DIN)
- new net: D95.2 (DOUT), D96.4 (DIN)
- new net: D49.2 (DOUT), D50.4 (DIN)
- new net: D30.2 (DOUT), D31.4 (DIN)
- new net: D29.2 (DOUT), D30.4 (DIN)
- new net: D52.2 (DOUT), D53.4 (DIN)
- new net: D190.4 (DIN), D192.2 (DOUT)
- new net: D112.2 (DOUT), D113.4 (DIN)
- new net: D78.2 (DOUT), D79.4 (DIN)
- new net: D144.4 (DIN), D146.2 (DOUT)
- new net: D175.2 (DOUT), D177.4 (DIN)
- new net: D208.4 (DIN), D210.2 (DOUT)
- new net: D210.4 (DIN), D212.2 (DOUT)
- new net: D230.4 (DIN), D232.2 (DOUT)
- new net: D232.4 (DIN), D234.2 (DOUT)
- new net: D142.4 (DIN), D144.2 (DOUT)
- new net: D58.2 (DOUT), D59.4 (DIN)
- new net: D57.2 (DOUT), D58.4 (DIN)
- new net: D165.2 (DOUT), D167.4 (DIN)
- new net: D23.2 (DOUT), D24.4 (DIN)
- new net: D196.4 (DIN), D198.2 (DOUT)
- new net: D186.4 (DIN), D188.2 (DOUT)
- new net: D188.4 (DIN), D190.2 (DOUT)
- new net: D24.2 (DOUT), D25.4 (DIN)
- new net: D135.2 (DOUT), D137.4 (DIN)
- new net: D133.2 (DOUT), D135.4 (DIN)
- new net: D150.4 (DIN), D152.2 (DOUT)
- new net: D152.4 (DIN), D154.2 (DOUT)
- new net: D180.4 (DIN), D182.2 (DOUT)
- new net: D61.2 (DOUT), D62.4 (DIN)
- new net: D60.2 (DOUT), D61.4 (DIN)
- new net: D245.2 (DOUT), D247.4 (DIN)
- new net: D243.2 (DOUT), D245.4 (DIN)
- new net: D158.4 (DIN), D160.2 (DOUT)
- new net: D160.4 (DIN), D162.2 (DOUT)
- new net: D54.2 (DOUT), D55.4 (DIN)
- new net: D53.2 (DOUT), D54.4 (DIN)
- new net: D74.2 (DOUT), D75.4 (DIN)
- new net: D73.2 (DOUT), D74.4 (DIN)
- new net: D81.2 (DOUT), D82.4 (DIN)
- new net: D70.2 (DOUT), D71.4 (DIN)
- new net: D94.2 (DOUT), D95.4 (DIN)
- new net: D218.4 (DIN), D220.2 (DOUT)
- new net: D59.2 (DOUT), D60.4 (DIN)
- new net: D28.2 (DOUT), D29.4 (DIN)
- new net: D174.4 (DIN), D176.2 (DOUT)
- new net: D48.2 (DOUT), D49.4 (DIN)
- new net: D246.4 (DIN), D248.2 (DOUT)
- new net: D248.4 (DIN), D250.2 (DOUT)
- new net: D145.2 (DOUT), D147.4 (DIN)
- new net: D116.2 (DOUT), D117.4 (DIN)
- new net: D115.2 (DOUT), D116.4 (DIN)
- new net: D217.2 (DOUT), D219.4 (DIN)
- new net: D215.2 (DOUT), D217.4 (DIN)
- new net: D122.2 (DOUT), D123.4 (DIN)
- new net: D84.2 (DOUT), D85.4 (DIN)
- new net: D72.2 (DOUT), D73.4 (DIN)
- new net: D182.4 (DIN), D184.2 (DOUT)
- new net: D204.4 (DIN), D206.2 (DOUT)
- new net: D206.4 (DIN), D208.2 (DOUT)
- new net: D64.2 (DOUT), D65.4 (DIN)
- new net: D227.2 (DOUT), D229.4 (DIN)
- new net: D117.2 (DOUT), D118.4 (DIN)
- new net: D250.4 (DIN), D252.2 (DOUT)
- new net: D252.4 (DIN), D254.2 (DOUT)
- new net: D154.4 (DIN), D156.2 (DOUT)
- new net: D128.2 (DOUT), D129.4 (DIN)
- new net: D92.2 (DOUT), D93.4 (DIN)
- new net: D91.2 (DOUT), D92.4 (DIN)
- new net: D202.4 (DIN), D204.2 (DOUT)
- new net: D71.2 (DOUT), D72.4 (DIN)
- new net: D123.2 (DOUT), D124.4 (DIN)
- new net: D80.2 (DOUT), D81.4 (DIN)
- new net: D101.2 (DOUT), D102.4 (DIN)
- new net: D79.2 (DOUT), D80.4 (DIN)
- new net: D97.2 (DOUT), D98.4 (DIN)
- new net: D90.2 (DOUT), D91.4 (DIN)
- new net: D25.2 (DOUT), D26.4 (DIN)
- new net: D225.2 (DOUT), D227.4 (DIN)
- new net: D223.2 (DOUT), D225.4 (DIN)
- new net: D184.4 (DIN), D186.2 (DOUT)
- new net: D42.2 (DOUT), D43.4 (DIN)
- new net: D153.2 (DOUT), D155.4 (DIN)
- new net: D93.2 (DOUT), D94.4 (DIN)
- new net: D224.4 (DIN), D226.2 (DOUT)
- new net: D187.2 (DOUT), D189.4 (DIN)
- new net: D185.2 (DOUT), D187.4 (DIN)
- new net: D221.2 (DOUT), D223.4 (DIN)
- new net: D138.4 (DIN), D140.2 (DOUT)
- new net: D140.4 (DIN), D142.2 (DOUT)
- new net: D173.2 (DOUT), D175.4 (DIN)
- new net: D209.2 (DOUT), D211.4 (DIN)
- new net: D167.2 (DOUT), D169.4 (DIN)
- new net: D31.2 (DOUT), D32.4 (DIN)
- new net: D85.2 (DOUT), D86.4 (DIN)
- new net: D156.4 (DIN), D158.2 (DOUT)
- new net: D100.2 (DOUT), D101.4 (DIN)
- new net: D104.2 (DOUT), D105.4 (DIN)
- new net: D39.2 (DOUT), D40.4 (DIN)
- new net: D114.2 (DOUT), D115.4 (DIN)
- new net: D34.2 (DOUT), D35.4 (DIN)
- new net: D211.2 (DOUT), D213.4 (DIN)
- new net: D247.2 (DOUT), D249.4 (DIN)
- new net: D43.2 (DOUT), D44.4 (DIN)
- new net: D119.2 (DOUT), D120.4 (DIN)
- new net: D118.2 (DOUT), D119.4 (DIN)
- new net: D181.2 (DOUT), D183.4 (DIN)
- new net: D193.2 (DOUT), D195.4 (DIN)
- new net: D141.2 (DOUT), D143.4 (DIN)
- new net: D213.2 (DOUT), D215.4 (DIN)
- new net: D183.2 (DOUT), D185.4 (DIN)
- new net: D236.4 (DIN), D238.2 (DOUT)
- new net: D164.4 (DIN), D166.2 (DOUT)
- new net: D162.4 (DIN), D164.2 (DOUT)
- new net: D113.2 (DOUT), D114.4 (DIN)
- new net: D234.4 (DIN), D236.2 (DOUT)
- new net: D143.2 (DOUT), D145.4 (DIN)
- new net: D109.2 (DOUT), D110.4 (DIN)
- new net: D219.2 (DOUT), D221.4 (DIN)
- new net: D151.2 (DOUT), D153.4 (DIN)
- new net: D36.2 (DOUT), D37.4 (DIN)
- new net: D35.2 (DOUT), D36.4 (DIN)
Other:
- moved on the sheet: TP1, TP2, TP3

Commit message: designing
Parts:
- added TP4, TP5, TP6: TestPoint, Pegoku:TestPoint, symbol Connector:TestPoint
Connections:
- net +5V: now also TP4.1
- net GND: now also TP5.1
Changed lines of the file:
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@@
 	)
 	(junction
+		(at -318.7432 59.69)
+		(diameter 0)
+		(color 0 0 0 0)
+	)
+	(junction
 		(at -204.47 29.21)
 		(diameter 0)
@@
 	)
 	(junction
+		(at -311.15 74.93)
+		(diameter 0)
+		(color 0 0 0 0)
+	)
+	(junction
 		(at 572.77 13.97)
 		(diameter 0)
@@
 	(wire
 		(pts
+			(xy -311.15 74.93) (xy -295.91 74.93)
+		)
+		(stroke
+			(width 0)
+			(type default)
+		)
+	)
+	(wire
+		(pts
 			(xy -158.75 13.97) (xy -143.51 13.97)
 		)
@@
 	(wire
 		(pts
+			(xy -318.7432 59.69) (xy -311.15 59.69)
+		)
+		(stroke
+			(width 0)
+			(type default)
+		)
+	)
+	(wire
+		(pts
 			(xy 328.93 13.97) (xy 344.17 13.97)
 		)
@@
 	(wire
 		(pts
+			(xy -318.77 74.93) (xy -311.15 74.93)
+		)
+		(stroke
+			(width 0)
+			(type default)
+		)
+	)
+	(wire
+		(pts
 			(xy -219.71 29.21) (xy -204.47 29.21)
 		)
@@
 	(wire
 		(pts
-			(xy -325.12 59.69) (xy -311.15 59.69)
+			(xy -325.12 59.69) (xy -318.7432 59.69)
 		)
 		(stroke
@@
 	(wire
 		(pts
-			(xy -295.91 74.93) (xy -311.15 74.93)
-		)
-		(stroke
-			(width 0)
-			(type default)
-		)
-	)
-	(wire
-		(pts
 			(xy 481.33 44.45) (xy 466.09 44.45)
 		)
@@
 	)
 	(symbol
+		(lib_id "Connector:TestPoint")
+		(at -318.7432 67.31 0)
+		(unit 1)
+		(exclude_from_sim no)
+		(in_bom yes)
+		(on_board yes)
+		(dnp no)
+		(property "Reference" "TP6"
+			(at -316.2032 62.7379 0)
+			(effects
+				(font
+					(size 1.27 1.27)
+				)
+				(justify left)
+			)
+		)
+		(property "Value" "TestPoint"
+			(at -316.2032 65.2779 0)
+			(effects
+				(font
+					(size 1.27 1.27)
+				)
+				(justify left)
+			)
+		)
+		(property "Footprint" "Pegoku:TestPoint"
+			(at -313.6632 67.31 0)
+			(effects
+				(font
+					(size 1.27 1.27)
+				)
+				(hide yes)
+			)
+		)
+		(property "Datasheet" "~"
+			(at -313.6632 67.31 0)
+			(effects
+				(font
+					(size 1.27 1.27)
+				)
+				(hide yes)
+			)
+		)
+		(property "Description" "test point"
+			(at -318.7432 67.31 0)
+			(effects
+				(font
+					(size 1.27 1.27)
+				)
+				(hide yes)
+			)
+		)
+		(pin "1"
+		)
+		(instances
+			(project "Neopixel"
+				(path "/0c64f9f6-2337-46e9-954e-fa62cdf10650"
+					(reference "TP6")
+					(unit 1)
+				)
+			)
+		)
+	)
+	(symbol
 		(lib_id "LED:WS2812B")
 		(at -6.35 36.83 180)
@@
 	)
 	(symbol
+		(lib_id "Connector:TestPoint")
+		(at -318.7432 59.69 0)
+		(unit 1)
+		(exclude_from_sim no)
+		(in_bom yes)
+		(on_board yes)
+		(dnp no)
+		(property "Reference" "TP5"
+			(at -316.2032 55.1179 0)
+			(effects
+				(font
+					(size 1.27 1.27)
+				)
+				(justify left)
+			)
+		)
+		(property "Value" "TestPoint"
+			(at -316.2032 57.6579 0)
+			(effects
+				(font
+					(size 1.27 1.27)
+				)
+				(justify left)
+			)
+		)
+		(property "Footprint" "Pegoku:TestPoint"
+			(at -313.6632 59.69 0)
+			(effects
+				(font
+					(size 1.27 1.27)
+				)
+				(hide yes)
+			)
+		)
+		(property "Datasheet" "~"
+			(at -313.6632 59.69 0)
+			(effects
+				(font
+					(size 1.27 1.27)
+				)
+				(hide yes)
+			)
+		)
+		(property "Description" "test point"
+			(at -318.7432 59.69 0)
+			(effects
+				(font
+					(size 1.27 1.27)
+				)
+				(hide yes)
+			)
+		)
+		(pin "1"
+		)
+		(instances
+			(project "Neopixel"
+				(path "/0c64f9f6-2337-46e9-954e-fa62cdf10650"
+					(reference "TP5")
+					(unit 1)
+				)
+			)
+		)
+	)
+	(symbol
 		(lib_id "LED:WS2812B")
 		(at -143.51 36.83 180)
@@
 					(unit 1)
 				)
+			)
+		)
+	)
+	(symbol
+		(lib_id "Connector:TestPoint")
+		(at -318.77 74.93 0)
+		(unit 1)
+		(exclude_from_sim no)
+		(in_bom yes)
+		(on_board yes)
+		(dnp no)
+		(property "Reference" "TP4"
+			(at -316.23 70.3579 0)
+			(effects
+				(font
+					(size 1.27 1.27)
+				)
+				(justify left)
+			)
+		)
+		(property "Value" "TestPoint"
+			(at -316.23 72.8979 0)
+			(effects
+				(font
+					(size 1.27 1.27)
+				)
+				(justify left)
+			)
+		)
+		(property "Footprint" "Pegoku:TestPoint"
+			(at -313.69 74.93 0)
+			(effects
+				(font
+					(size 1.27 1.27)
+				)
+				(hide yes)
+			)
+		)
+		(property "Datasheet" "~"
+			(at -313.69 74.93 0)
+			(effects
+				(font
+					(size 1.27 1.27)
+				)
+				(hide yes)
+			)
+		)
+		(property "Description" "test point"
+			(at -318.77 74.93 0)
+			(effects
+				(font
+					(size 1.27 1.27)
+				)
+				(hide yes)
+			)
+		)
+		(pin "1"
+		)
+		(instances
+			(project "Neopixel"
+				(path "/0c64f9f6-2337-46e9-954e-fa62cdf10650"
+					(reference "TP4")
+					(unit 1)
+				)

Commit message: designing
Parts:
- removed TP4, TP5, TP6: TestPoint, Pegoku:TestPoint, symbol Connector:TestPoint
Connections:
- net at D193.4 (DIN): now also D194.2 (DOUT); no longer D191.2 (DOUT)
- net at D189.2 (DOUT): now also D190.4 (DIN); no longer D191.4 (DIN)
- net at D130.4 (DIN): now also D129.2 (DOUT); no longer D132.2 (DOUT)
- net at D134.2 (DOUT): now also D135.4 (DIN); no longer D132.4 (DIN)
- net at D203.2 (DOUT): now also D202.4 (DIN); no longer D205.4 (DIN)
- net at D201.2 (DOUT): now also D200.4 (DIN); no longer D203.4 (DIN)
- net at D242.4 (DIN): now also D243.2 (DOUT); no longer D244.2 (DOUT)
- net at D244.4 (DIN): now also D245.2 (DOUT); no longer D246.2 (DOUT)
- net at D159.4 (DIN): now also D158.2 (DOUT); no longer D157.2 (DOUT)
- net at D155.2 (DOUT): now also D156.4 (DIN); no longer D157.4 (DIN)
- net at D148.2 (DOUT): now also D149.4 (DIN); no longer D146.4 (DIN)
- net at D150.2 (DOUT): now also D151.4 (DIN); no longer D148.4 (DIN)
- net at D199.4 (DIN): now also D200.2 (DOUT); no longer D197.2 (DOUT)
- net at D195.2 (DOUT): now also D194.4 (DIN); no longer D197.4 (DIN)
- net at D166.4 (DIN): now also D165.2 (DOUT); no longer D168.2 (DOUT)
- net at D168.4 (DIN): now also D167.2 (DOUT); no longer D170.2 (DOUT)
- net at D243.4 (DIN): now also D244.2 (DOUT); no longer D241.2 (DOUT)
- net at D241.4 (DIN): now also D242.2 (DOUT); no longer D239.2 (DOUT)
- net at D214.4 (DIN): now also D215.2 (DOUT); no longer D216.2 (DOUT)
- net at D218.2 (DOUT): now also D217.4 (DIN); no longer D216.4 (DIN)
- net at D233.4 (DIN): now also D234.2 (DOUT); no longer D231.2 (DOUT)
- net at D229.2 (DOUT): now also D228.4 (DIN); no longer D231.4 (DIN)
- net at D214.2 (DOUT): now also D213.4 (DIN); no longer D212.4 (DIN)
- net at D176.4 (DIN): now also D175.2 (DOUT); no longer D178.2 (DOUT)
- net at D180.2 (DOUT): now also D181.4 (DIN); no longer D178.4 (DIN)
- net at D198.4 (DIN): now also D199.2 (DOUT); no longer D200.2 (DOUT)
- net at D202.2 (DOUT): now also D201.4 (DIN); no longer D200.4 (DIN)
- net at D134.4 (DIN): now also D133.2 (DOUT); no longer D136.2 (DOUT)
- net at D138.2 (DOUT): now also D139.4 (DIN); no longer D136.4 (DIN)
- net at D238.4 (DIN): now also D239.2 (DOUT); no longer D240.2 (DOUT)
- net at D240.4 (DIN): now also D241.2 (DOUT); no longer D242.2 (DOUT)
- net at D235.4 (DIN): now also D236.2 (DOUT); no longer D233.2 (DOUT)
- net at D141.4 (DIN): now also D140.2 (DOUT); no longer D139.2 (DOUT)
- net at D137.2 (DOUT): now also D138.4 (DIN); no longer D139.4 (DIN)
- net at D179.2 (DOUT): now also D180.4 (DIN); no longer D181.4 (DIN)
- net at D177.2 (DOUT): now also D178.4 (DIN); no longer D179.4 (DIN)
- net at D133.4 (DIN): now also D132.2 (DOUT); no longer D131.2 (DOUT)
- net at D131.4 (DIN): now also D130.2 (DOUT); no longer D129.2 (DOUT)
- net at D255.4 (DIN): now also D256.2 (DOUT); no longer D253.2 (DOUT)
- net at D253.4 (DIN): now also D254.2 (DOUT); no longer D251.2 (DOUT)
- net at D251.4 (DIN): now also D252.2 (DOUT); no longer D249.2 (DOUT)
- net at D209.4 (DIN): now also D210.2 (DOUT); no longer D207.2 (DOUT)
- net at D205.2 (DOUT): now also D204.4 (DIN); no longer D207.4 (DIN)
- net at D192.4 (DIN): now also D191.2 (DOUT); no longer D194.2 (DOUT)
- net at D196.2 (DOUT): now also D195.4 (DIN); no longer D194.4 (DIN)
- net at D254.4 (DIN): now also D255.2 (DOUT); no longer D256.2 (DOUT)
- net at D256.4 (DIN): no longer D255.2 (DOUT)
- net at D165.4 (DIN): now also D164.2 (DOUT); no longer D163.2 (DOUT)
- net at D161.2 (DOUT): now also D162.4 (DIN); no longer D163.4 (DIN)
- net at D220.4 (DIN): now also D221.2 (DOUT); no longer D222.2 (DOUT)
- net at D222.4 (DIN): now also D223.2 (DOUT); no longer D224.2 (DOUT)
- net at D173.4 (DIN): now also D172.2 (DOUT); no longer D171.2 (DOUT)
- net at D169.2 (DOUT): now also D170.4 (DIN); no longer D171.4 (DIN)
- net at D228.2 (DOUT): now also D227.4 (DIN); no longer D226.4 (DIN)
- net at D230.2 (DOUT): now also D229.4 (DIN); no longer D228.4 (DIN)
- net at D161.4 (DIN): now also D160.2 (DOUT); no longer D159.2 (DOUT)
- net at D149.2 (DOUT): now also D150.4 (DIN); no longer D151.4 (DIN)
- net at D147.2 (DOUT): now also D148.4 (DIN); no longer D149.4 (DIN)
- net at D239.4 (DIN): now also D240.2 (DOUT); no longer D237.2 (DOUT)
- net at D235.2 (DOUT): now also D234.4 (DIN); no longer D237.4 (DIN)
- net at D174.2 (DOUT): now also D175.4 (DIN); no longer D172.4 (DIN)
- net at D192.2 (DOUT): now also D193.2 (DOUT); no longer D190.4 (DIN)
- net at D144.4 (DIN): now also D143.2 (DOUT); no longer D146.2 (DOUT)
- net at D177.4 (DIN): now also D176.2 (DOUT); no longer D175.2 (DOUT)
- net at D208.4 (DIN): now also D209.2 (DOUT); no longer D210.2 (DOUT)
- net at D210.4 (DIN): now also D211.2 (DOUT); no longer D212.2 (DOUT)
- net at D230.4 (DIN): now also D231.2 (DOUT); no longer D232.2 (DOUT)
- net at D232.4 (DIN): now also D233.2 (DOUT); no longer D234.2 (DOUT)
- net at D144.2 (DOUT): now also D145.4 (DIN); no longer D142.4 (DIN)
- net at D167.4 (DIN): now also D166.2 (DOUT); no longer D165.2 (DOUT)
- net at D198.2 (DOUT): now also D197.4 (DIN); no longer D196.4 (DIN)
- net at D186.4 (DIN): now also D185.2 (DOUT); no longer D188.2 (DOUT)
- net at D188.4 (DIN): now also D187.2 (DOUT); no longer D190.2 (DOUT)
- net at D137.4 (DIN): now also D136.2 (DOUT); no longer D135.2 (DOUT)
- net at D152.2 (DOUT): now also D153.4 (DIN); no longer D150.4 (DIN)
- net at D152.4 (DIN): now also D151.2 (DOUT); no longer D154.2 (DOUT)
- net at D182.2 (DOUT): now also D183.4 (DIN); no longer D180.4 (DIN)
- net at D247.4 (DIN): now also D248.2 (DOUT); no longer D245.2 (DOUT)
- net at D245.4 (DIN): now also D246.2 (DOUT); no longer D243.2 (DOUT)
- net at D158.4 (DIN): now also D157.2 (DOUT); no longer D160.2 (DOUT)
- net at D162.2 (DOUT): now also D163.4 (DIN); no longer D160.4 (DIN)
- net at D218.4 (DIN): now also D219.2 (DOUT); no longer D220.2 (DOUT)
- net at D174.4 (DIN): now also D173.2 (DOUT); no longer D176.2 (DOUT)
- net at D246.4 (DIN): now also D247.2 (DOUT); no longer D248.2 (DOUT)
- net at D250.2 (DOUT): now also D249.4 (DIN); no longer D248.4 (DIN)
- net at D145.2 (DOUT): now also D146.4 (DIN); no longer D147.4 (DIN)
- net at D219.4 (DIN): now also D220.2 (DOUT); no longer D217.2 (DOUT)
- net at D184.2 (DOUT): now also D185.4 (DIN); no longer D182.4 (DIN)
- net at D206.2 (DOUT): now also D205.4 (DIN); no longer D204.4 (DIN)
- net at D206.4 (DIN): now also D207.2 (DOUT); no longer D208.2 (DOUT)
- net at D227.2 (DOUT): now also D226.4 (DIN); no longer D229.4 (DIN)
- net at D250.4 (DIN): now also D251.2 (DOUT); no longer D252.2 (DOUT)
- net at D252.4 (DIN): now also D253.2 (DOUT); no longer D254.2 (DOUT)
- net at D154.4 (DIN): now also D153.2 (DOUT); no longer D156.2 (DOUT)
- net at D204.2 (DOUT): now also D203.4 (DIN); no longer D202.4 (DIN)
- net at D225.2 (DOUT): now also D224.4 (DIN); no longer D227.4 (DIN)
- net at D225.4 (DIN): now also D226.2 (DOUT); no longer D223.2 (DOUT)
- net at D184.4 (DIN): now also D183.2 (DOUT); no longer D186.2 (DOUT)
- net at D155.4 (DIN): now also D154.2 (DOUT); no longer D153.2 (DOUT)
- net at D189.4 (DIN): now also D188.2 (DOUT); no longer D187.2 (DOUT)
- net at D187.4 (DIN): now also D186.2 (DOUT); no longer D185.2 (DOUT)
- net at D223.4 (DIN): now also D224.2 (DOUT); no longer D221.2 (DOUT)
- net at D142.2 (DOUT): now also D143.4 (DIN); no longer D140.4 (DIN)
- net at D211.4 (DIN): now also D212.2 (DOUT); no longer D209.2 (DOUT)
- net at D169.4 (DIN): now also D168.2 (DOUT); no longer D167.2 (DOUT)
- net at D181.2 (DOUT): now also D182.4 (DIN); no longer D183.4 (DIN)
- net at D141.2 (DOUT): now also D142.4 (DIN); no longer D143.4 (DIN)
- net at D215.4 (DIN): now also D216.2 (DOUT); no longer D213.2 (DOUT)
- net at D238.2 (DOUT): now also D237.4 (DIN); no longer D236.4 (DIN)
- net at D164.4 (DIN): now also D163.2 (DOUT); no longer D166.2 (DOUT)
- net at D221.4 (DIN): now also D222.2 (DOUT); no longer D219.2 (DOUT)
- new net: D231.4 (DIN), D232.2 (DOUT)
- new net: D216.4 (DIN), D217.2 (DOUT)
- new net: D212.4 (DIN), D213.2 (DOUT)
- new net: D135.2 (DOUT), D136.4 (DIN)
- new net: D156.2 (DOUT), D157.4 (DIN)
- new net: D139.2 (DOUT), D140.4 (DIN)
- new net: D171.2 (DOUT), D172.4 (DIN)
- new net: D248.4 (DIN), D249.2 (DOUT)
- new net: D236.4 (DIN), D237.2 (DOUT)
- new net: D207.4 (DIN), D208.2 (DOUT)
- new net: D146.2 (DOUT), D147.4 (DIN)
- new net: D196.4 (DIN), D197.2 (DOUT)
- new net: D159.2 (DOUT), D160.4 (DIN)
- new net: D178.2 (DOUT), D179.4 (DIN)
- new net: D131.2 (DOUT), D132.4 (DIN)
- new net: D170.2 (DOUT), D171.4 (DIN)
- new net: D190.2 (DOUT), D191.4 (DIN)
